Commit message: Updated puzzlebot_controller.yaml

File: puzzlebot_description/urdf/puzzlebot.urdf.xacro (robot description, xacro)
@@ -5,4 +5,10 @@
   <!-- Include ros2_control Plugins -->
   <xacro:include filename="$(find puzzlebot_description)/urdf/puzzlebot_ros2_control.xacro"/>
+  <link name="world"/>  <!-- Gazebo's global fixed frame -->
+  <joint name="world_to_base_joint" type="fixed">
+    <parent link="world"/>
+    <child link="base_link"/>
+    <origin xyz="0 0 0.025" rpy="0 0 0"/>
+  </joint>
   <link
     name="base_link">
@@ -120,5 +126,5 @@
         name="">
         <color
-          rgba="1 1 1 0.35" />
+          rgba="0 0 0 1" />
       </material>
     </visual>
@@ -174,5 +180,5 @@
         name="">
         <color
-          rgba="1 1 1 0.35" />
+          rgba="0 0 0 1" />
       </material>
     </visual>

File: puzzlebot_description/urdf/puzzlebot_ros2_control.xacro (robot description, xacro)
@@ -2,10 +2,7 @@
 <robot xmlns:xacro="http://ros.org/wiki/xacro">
     <ros2_control type="system" name="RobotSystem">
-        <!-- <hardware>
-            <plugin>gz_ros2_control/GazeboSimSystem</plugin>
-        </hardware> -->
         <hardware>
             <plugin>ign_ros2_control/IgnitionSystem</plugin>
-            <param name="use_sim_time">true</param>  /this one works
+            <param name="use_sim_time">true</param>
         </hardware>
         <!-- Define the wheel joints and control interfaces -->

Commit message: Update puzzlebot_description

File: puzzlebot_description/urdf/puzzlebot.urdf.xacro (robot description, xacro)
@@ -4,10 +4,11 @@
   <xacro:include filename="$(find puzzlebot_description)/urdf/puzzlebot_gazebo.xacro"/>
   <!-- Include ros2_control Plugins -->
-  <xacro:include filename="$(find puzzlebot_description)/urdf/puzzlebot_ros2_control.xacro"/>
-  <link name="world"/>  <!-- Gazebo's global fixed frame -->
-  <joint name="world_to_base_joint" type="fixed">
-    <parent link="world"/>
+  <!-- <xacro:include filename="$(find puzzlebot_description)/urdf/puzzlebot_ros2_control.xacro"/> -->
+  <!-- Add this near the top of your URDF, after <robot> tag -->
+  <link name="odom"/>
+  <joint name="odom_joint" type="fixed">
+    <parent link="odom"/>
     <child link="base_link"/>
-    <origin xyz="0 0 0.025" rpy="0 0 0"/>
+    <origin xyz="0 0 0" rpy="0 0 0"/>
   </joint>
   <link
@@ -49,5 +50,5 @@
     </collision>
   </link>
-  <link
+  <!-- <link
     name="caster_link">
     <inertial>
@@ -99,5 +100,5 @@
     <axis
       xyz="0 0 0" />
-  </joint>
+  </joint> -->
   <link
     name="wheel_R_link">
@@ -151,6 +152,6 @@
       xyz="0 1 0" />
     <limit
-      effort="3"
-      velocity="0.5" />
+      effort="0.5"
+      velocity="5.0" />
   </joint>
   <link
@@ -203,8 +204,27 @@
       link="wheel_L_link" />
     <axis
-      xyz="0 -1 0" />
+      xyz="0 1 0" />
     <limit
-      effort="3"
-      velocity="0.5" />
+      effort="0.5"
+      velocity="5.0" />
+  </joint>
+  <link name="camera_link">
+    <visual>
+        <geometry>
+            <box size="0.020 0.020 0.020"/> <!-- Simple box for visualization -->
+        </geometry>
+        <material name="blue">
+            <color rgba="0 0 0.8 1"/>
+        </material>
+    </visual>
+    <inertial>
+        <mass value="0.01"/>
+        <inertia ixx="0.001" ixy="0.0" ixz="0.0" iyy="0.001" iyz="0.0" izz="0.001"/>
+    </inertial>
+  </link>
+  <joint name="camera_joint" type="fixed">
+      <parent link="base_link"/>
+      <child link="camera_link"/>
+      <origin xyz="0.04 0 0.06" rpy="0 0 0"/> <!-- Adjust position as needed -->
   </joint>
 </robot>

File: puzzlebot_description/urdf/puzzlebot_gazebo.xacro (robot description, xacro)
@@ -1,9 +1,62 @@
 <?xml version="1.0"?>
-<robot xmlns:xacro="http://wiki.ros.org/xacro">
-    <gazebo>
-        <plugin filename="ign_ros2_control-system" name="ign_ros2_control::IgnitionROS2ControlPlugin">
-            <parameters>$(find puzzlebot_description)/config/puzzlebot_controller.yaml</parameters>
-            <topic>/model/puzzlebot/cmd_vel</topic>
-        </plugin>
-    </gazebo>
+<robot xmlns:xacro="http://www.ros.org/wiki/xacro">
+  <!-- Differential Drive Plugin -->
+  <gazebo>
+    <plugin filename="libignition-gazebo-diff-drive-system.so" name="ignition::gazebo::systems::DiffDrive">
+      <left_joint>wheel_L_joint</left_joint>
+      <right_joint>wheel_R_joint</right_joint>
+      <wheel_separation>0.181</wheel_separation>
+      <wheel_radius>0.05</wheel_radius>
+      <!-- <wheel_radius>0.03045</wheel_radius>        -->
+      <topic>cmd_vel</topic>
+      <odom_topic>odom</odom_topic>
+      <odom_frame>odom</odom_frame>
+      <robot_base_frame>base_link</robot_base_frame>
+      <publish_odom>true</publish_odom>
+      <publish_odom_tf>true</publish_odom_tf>
+      <min_velocity>-5.0</min_velocity>
+      <max_velocity>5.0</max_velocity>
+      <min_acceleration>-10.0</min_acceleration>
+      <max_acceleration>10.0</max_acceleration>
+    </plugin>
+  </gazebo>
+  <!-- Wheel friction coefficients -->
+  <!-- <gazebo reference="wheel_L_link">
+    <mu1>0.8</mu1>
+    <mu2>0.8</mu2>
+    <kp>100000.0</kp>
+    <kd>10.0</kd>
+  </gazebo>
+  <gazebo reference="wheel_R_link">
+    <mu1>0.8</mu1>
+    <mu2>0.8</mu2>
+    <kp>100000.0</kp>
+    <kd>10.0</kd>
+  </gazebo> -->
+  <gazebo reference="wheel_R_link">
+    <mu1>100000000000000.0</mu1>
+    <mu2>100000000000000.0</mu2>
+    <kp>1000000000000.0</kp>
+    <kd>10.0</kd>
+    <minDepth>0.001</minDepth>
+    <maxVel>0.1</maxVel>
+    <fdir1>0 1 0</fdir1>
+  </gazebo>
+  <gazebo reference="wheel_L_link">
+    <mu1>100000000000000.0</mu1>
+    <mu2>100000000000000.0</mu2>
+    <kp>1000000000000.0</kp>
+    <kd>10.0</kd>
+    <minDepth>0.001</minDepth>
+    <maxVel>0.1</maxVel>
+    <fdir1>0 1 0</fdir1>
+  </gazebo>
+  <!-- <gazebo reference="caster_link">
+    <mu1>0.1</mu1>
+    <mu2>0.1</mu2>
+    <kp>1000000.0</kp>
+    <kd>100.0</kd>
+    <minDepth>0.001</minDepth>
+    <maxVel>0.1</maxVel>
+  </gazebo> -->
 </robot>

Commit message: New pkg

File: puzzlebot_description/urdf/puzzlebot.urdf.xacro (robot description, xacro)
@@ -3,13 +3,5 @@
   <!-- Include Gazebo Parameters -->
   <xacro:include filename="$(find puzzlebot_description)/urdf/puzzlebot_gazebo.xacro"/>
-  <!-- Include ros2_control Plugins -->
-  <!-- <xacro:include filename="$(find puzzlebot_description)/urdf/puzzlebot_ros2_control.xacro"/> -->
-  <!-- Add this near the top of your URDF, after <robot> tag -->
-  <link name="odom"/>
-  <joint name="odom_joint" type="fixed">
-    <parent link="odom"/>
-    <child link="base_link"/>
-    <origin xyz="0 0 0" rpy="0 0 0"/>
-  </joint>
+  <!-- <xacro:include filename="$(find puzzlebot_description)/urdf/p.xacro"/> -->
   <link
     name="base_link">

File: puzzlebot_description/urdf/puzzlebot_gazebo.xacro (robot description, xacro)
@@ -22,5 +22,5 @@
   </gazebo>
   <!-- Wheel friction coefficients -->
-  <!-- <gazebo reference="wheel_L_link">
+  <gazebo reference="wheel_L_link">
     <mu1>0.8</mu1>
     <mu2>0.8</mu2>
@@ -33,6 +33,6 @@
     <kp>100000.0</kp>
     <kd>10.0</kd>
-  </gazebo> -->
-  <gazebo reference="wheel_R_link">
+  </gazebo>
+  <!-- <gazebo reference="wheel_R_link">
     <mu1>100000000000000.0</mu1>
     <mu2>100000000000000.0</mu2>
@@ -51,5 +51,5 @@
     <maxVel>0.1</maxVel>
     <fdir1>0 1 0</fdir1>
-  </gazebo>
+  </gazebo> -->
   <!-- <gazebo reference="caster_link">
     <mu1>0.1</mu1>
